Commit message: Update ar_gripper_macro.xacro

File: annin_ar4_description/urdf/ar_gripper_macro.xacro (robot description, xacro)
@@ -13,5 +13,5 @@
       <visual>
         <geometry>
-          <mesh filename="file://$(find annin_ar4_description)/meshes/ar4_gripper/gripper_base_link.stl" />
+          <mesh filename="file://$(find annin_ar4_description)/meshes/ar4_mk3/spraygun_EE.stl" />
         </geometry>
         <material name="">

Commit message: Update ar_gripper_macro.xacro

File: annin_ar4_description/urdf/ar_gripper_macro.xacro (robot description, xacro)
@@ -1,3 +1,2 @@
-<?xml version="1.0" encoding="utf-8"?>
 <robot xmlns:xacro="http://wiki.ros.org/xacro">
   <xacro:macro name="ar_gripper" params="
@@ -21,5 +20,5 @@
       <collision>
         <geometry>
-          <mesh filename="file://$(find annin_ar4_description)/meshes/ar4_gripper/gripper_base_link.stl" />
+          <mesh filename="file://$(find annin_ar4_description)/meshes/ar4_mk3/spraygun_EE.stl" />
         </geometry>
       </collision>
@@ -30,59 +29,6 @@
       </inertial>
     </link>
-    <link name="${tf_prefix}gripper_jaw1_link">
-      <visual>
-        <geometry>
-          <mesh filename="file://$(find annin_ar4_description)/meshes/ar4_gripper/gripper_jaw1_link.stl" />
-        </geometry>
-        <material name="">
-          <color rgba="1 1 0 1"/>
-        </material>
-      </visual>
-      <collision>
-        <geometry>
-          <mesh filename="file://$(find annin_ar4_description)/meshes/ar4_gripper/gripper_jaw1_link.stl" />
-        </geometry>
-      </collision>
-      <inertial>
-        <origin xyz="-0.00435839 -0.00469536 0.00757141"/>
-        <mass value="0.01"/>
-        <inertia ixx="0.00000123" ixy="-0.00000004" ixz="0.00000012" iyy="0.00000115" iyz="0.00000016" izz="0.00000102"/>
-      </inertial>
-    </link>
-    <link name="${tf_prefix}gripper_jaw2_link">
-      <visual>
-        <geometry>
-          <mesh filename="file://$(find annin_ar4_description)/meshes/ar4_gripper/gripper_jaw2_link.stl" />
-        </geometry>
-        <material name="">
-          <color rgba="1 1 0 1"/>
-        </material>
-      </visual>
-      <collision>
-        <geometry>
-          <mesh filename="file://$(find annin_ar4_description)/meshes/ar4_gripper/gripper_jaw2_link.stl" />
-        </geometry>
-      </collision>
-      <inertial>
-        <origin xyz="-0.00423971 -0.00491236 0.00814582"/>
-        <mass value="0.01"/>
-        <inertia ixx="0.00000118" ixy="-0.00000004" ixz="0.00000013" iyy="0.00000110" iyz="0.00000013" izz="0.00000101"/>
-      </inertial>
-    </link>
-    <joint name="${tf_prefix}gripper_jaw1_joint" type="prismatic">
-      <origin xyz="0.0 -0.036 0" rpy="0.0 0.0 0.0"/>
-      <parent link="${tf_prefix}gripper_base_link"/>
-      <child link="${tf_prefix}gripper_jaw1_link"/>
-      <axis xyz="-1 0 0"/>
-      <limit lower="0" upper="0.014" effort="-1" velocity="1.0"/>
-    </joint>
-    <joint name="${tf_prefix}gripper_jaw2_joint" type="prismatic">
-      <origin xyz="0.0 -0.036 0" rpy="0.0 ${-pi} 0.0"/>
-      <parent link="${tf_prefix}gripper_base_link"/>
-      <child link="${tf_prefix}gripper_jaw2_link"/>
-      <axis xyz="-1 0 0"/>
-      <limit lower="0" upper="0.014" effort="1000" velocity="1.0"/>
-      <mimic joint="${tf_prefix}gripper_jaw1_joint" multiplier="1" offset="0"/>
-    </joint>
+    <!-- Remove gripper jaws and their joints -->
+    <!-- No need for gripper_jaw1_link, gripper_jaw2_link, or their respective joints -->
   </xacro:macro>
 </robot>

Commit message: Update ar_gripper_macro.xacro

File: annin_ar4_description/urdf/ar_gripper_macro.xacro (robot description, xacro)
@@ -1,7 +1,6 @@
+<?xml version="1.0"?>
 <robot xmlns:xacro="http://wiki.ros.org/xacro">
-  <xacro:macro name="ar_gripper" params="
-    tf_prefix
-    parent
-  ">
+  <xacro:macro name="ar_gripper" params="tf_prefix parent">
+    <!-- 固定ジョイントでエンドエフェクタに取り付け -->
     <joint name="${tf_prefix}gripper_base_joint" type="fixed">
       <origin xyz="0.0 0.0 0.0" rpy="-1.5708 0.0 0.0"/>
@@ -9,8 +8,11 @@
       <child link="${tf_prefix}gripper_base_link"/>
     </joint>
+    <!-- グリッパー本体（スプレーガン） -->
     <link name="${tf_prefix}gripper_base_link">
       <visual>
         <geometry>
-          <mesh filename="file://$(find annin_ar4_description)/meshes/ar4_mk3/spraygun_EE.stl" />
+          <mesh filename="file://$(find annin_ar4_description)/meshes/ar4_mk3/spraygun_EE.stl">
+            <scale>0.001 0.001 0.001</scale>
+          </mesh>
         </geometry>
         <material name="">
@@ -20,5 +22,7 @@
       <collision>
         <geometry>
-          <mesh filename="file://$(find annin_ar4_description)/meshes/ar4_mk3/spraygun_EE.stl" />
+          <mesh filename="file://$(find annin_ar4_description)/meshes/ar4_mk3/spraygun_EE.stl">
+            <scale>0.001 0.001 0.001</scale>
+          </mesh>
         </geometry>
       </collision>
@@ -26,9 +30,10 @@
         <origin xyz="-0.00073621 -0.02341392 -0.00435302"/>
         <mass value="0.08"/>
-        <inertia ixx="0.00002375" ixy="0.00000002" ixz="-0.00000017" iyy="0.00004082" iyz="-0.00000029" izz="0.00004254"/>
+        <inertia
+          ixx="0.00002375" ixy="0.00000002" ixz="-0.00000017"
+          iyy="0.00004082" iyz="-0.00000029" izz="0.00004254"/>
       </inertial>
     </link>
-    <!-- Remove gripper jaws and their joints -->
-    <!-- No need for gripper_jaw1_link, gripper_jaw2_link, or their respective joints -->
+    <!-- jaws（顎）や可動ジョイントは削除済み -->
   </xacro:macro>
 </robot>

Commit message: Update ar_gripper_macro.xacro

File: annin_ar4_description/urdf/ar_gripper_macro.xacro (robot description, xacro)
@@ -28,9 +28,8 @@
       </collision>
       <inertial>
-        <origin xyz="-0.00073621 -0.02341392 -0.00435302"/>
-        <mass value="0.08"/>
-        <inertia
-          ixx="0.00002375" ixy="0.00000002" ixz="-0.00000017"
-          iyy="0.00004082" iyz="-0.00000029" izz="0.00004254"/>
+        <origin xyz="0 0 0" rpy="0 0 0"/>
+        <mass value="1.5"/>
+        <inertia ixx="0.001" ixy="0" ixz="0"
+                 iyy="0.001" iyz="0" izz="0.001"/>
       </inertial>
     </link>

Commit message: Update ar_gripper_macro.xacro

File: annin_ar4_description/urdf/ar_gripper_macro.xacro (robot description, xacro)
@@ -12,7 +12,5 @@
       <visual>
         <geometry>
-          <mesh filename="file://$(find annin_ar4_description)/meshes/ar4_mk3/spraygun_EE.stl">
-            <scale>0.001 0.001 0.001</scale>
-          </mesh>
+          <mesh filename="file://$(find annin_ar4_description)/meshes/ar4_mk3/spraygun_EE.stl" scale="0.001 0.001 0.001"/>
         </geometry>
         <material name="">
@@ -22,7 +20,5 @@
       <collision>
         <geometry>
-          <mesh filename="file://$(find annin_ar4_description)/meshes/ar4_mk3/spraygun_EE.stl">
-            <scale>0.001 0.001 0.001</scale>
-          </mesh>
+          <mesh filename="file://$(find annin_ar4_description)/meshes/ar4_mk3/spraygun_EE.stl" scale="0.001 0.001 0.001"/>
         </geometry>
       </collision>
@@ -34,5 +30,4 @@
       </inertial>
     </link>
-    <!-- jaws（顎）や可動ジョイントは削除済み -->
   </xacro:macro>
 </robot>

Commit message: Update ar_gripper_macro.xacro

File: annin_ar4_description/urdf/ar_gripper_macro.xacro (robot description, xacro)
@@ -24,5 +24,5 @@
       </collision>
       <inertial>
-        <origin xyz="0 0 0" rpy="0 0 0"/>
+        <origin xyz="0 0 0" rpy="1.5708 0 0"/>
         <mass value="1.5"/>
         <inertia ixx="0.001" ixy="0" ixz="0"

Commit message: Update ar_gripper_macro.xacro

File: annin_ar4_description/urdf/ar_gripper_macro.xacro (robot description, xacro)
@@ -24,5 +24,5 @@
       </collision>
       <inertial>
-        <origin xyz="0 0 0" rpy="1.5708 0 0"/>
+        <origin xyz="0 0 0" rpy="1.5708 0 1.5708"/>
         <mass value="1.5"/>
         <inertia ixx="0.001" ixy="0" ixz="0"

Commit message: Update ar_gripper_macro.xacro

File: annin_ar4_description/urdf/ar_gripper_macro.xacro (robot description, xacro)
@@ -2,11 +2,11 @@
 <robot xmlns:xacro="http://wiki.ros.org/xacro">
   <xacro:macro name="ar_gripper" params="tf_prefix parent">
-    <!-- 固定ジョイントでエンドエフェクタに取り付け -->
+    <!-- エンドエフェクタに取り付け（Z→X回転） -->
     <joint name="${tf_prefix}gripper_base_joint" type="fixed">
-      <origin xyz="0.0 0.0 0.0" rpy="-1.5708 0.0 0.0"/>
+      <origin xyz="0.0 0.0 0.0" rpy="1.5708 0.0 1.5708"/>
       <parent link="${parent}"/>
       <child link="${tf_prefix}gripper_base_link"/>
     </joint>
-    <!-- グリッパー本体（スプレーガン） -->
+    <!-- スプレーガン本体 -->
     <link name="${tf_prefix}gripper_base_link">
       <visual>
@@ -24,5 +24,5 @@
       </collision>
       <inertial>
-        <origin xyz="0 0 0" rpy="1.5708 0 1.5708"/>
+        <origin xyz="0 0 0" rpy="0 0 0"/>
         <mass value="1.5"/>
         <inertia ixx="0.001" ixy="0" ixz="0"

Commit message: Update ar_gripper_macro.xacro

File: annin_ar4_description/urdf/ar_gripper_macro.xacro (robot description, xacro)
@@ -4,5 +4,5 @@
     <!-- エンドエフェクタに取り付け（Z→X回転） -->
     <joint name="${tf_prefix}gripper_base_joint" type="fixed">
-      <origin xyz="0.0 0.0 0.0" rpy="1.5708 0.0 1.5708"/>
+      <origin xyz="0.0 0.0 0.0" rpy="1.5708 0.0 0.0"/>
       <parent link="${parent}"/>
       <child link="${tf_prefix}gripper_base_link"/>

Commit message: Update ar_gripper_macro.xacro

File: annin_ar4_description/urdf/ar_gripper_macro.xacro (robot description, xacro)
@@ -4,5 +4,5 @@
     <!-- エンドエフェクタに取り付け（Z→X回転） -->
     <joint name="${tf_prefix}gripper_base_joint" type="fixed">
-      <origin xyz="0.0 0.0 0.0" rpy="1.5708 0.0 0.0"/>
+      <origin xyz="0.0 0.0 0.0" rpy="0.0 1.5708 0.0"/>
       <parent link="${parent}"/>
       <child link="${tf_prefix}gripper_base_link"/>

Commit message: Update ar_gripper_macro.xacro

File: annin_ar4_description/urdf/ar_gripper_macro.xacro (robot description, xacro)
@@ -4,5 +4,5 @@
     <!-- エンドエフェクタに取り付け（Z→X回転） -->
     <joint name="${tf_prefix}gripper_base_joint" type="fixed">
-      <origin xyz="0.0 0.0 0.0" rpy="0.0 1.5708 0.0"/>
+      <origin xyz="0.0 0.0 0.0" rpy="${pi} 0 ${-pi/2}">
       <parent link="${parent}"/>
       <child link="${tf_prefix}gripper_base_link"/>

Commit message: Update ar_gripper_macro.xacro

File: annin_ar4_description/urdf/ar_gripper_macro.xacro (robot description, xacro)
@@ -4,5 +4,5 @@
     <!-- エンドエフェクタに取り付け（Z→X回転） -->
     <joint name="${tf_prefix}gripper_base_joint" type="fixed">
-      <origin xyz="0.0 0.0 0.0" rpy="${pi} 0 ${-pi/2}">
+      <origin xyz="0.0 0.0 0.0" rpy="${pi} 0 ${-pi/2}"/>  <!-- ← タグを正しく閉じた -->
       <parent link="${parent}"/>
       <child link="${tf_prefix}gripper_base_link"/>
@@ -12,5 +12,6 @@
       <visual>
         <geometry>
-          <mesh filename="file://$(find annin_ar4_description)/meshes/ar4_mk3/spraygun_EE.stl" scale="0.001 0.001 0.001"/>
+          <mesh filename="file://$(find annin_ar4_description)/meshes/ar4_mk3/spraygun_EE.stl"
+                scale="0.001 0.001 0.001"/>
         </geometry>
         <material name="">
@@ -20,5 +21,6 @@
       <collision>
         <geometry>
-          <mesh filename="file://$(find annin_ar4_description)/meshes/ar4_mk3/spraygun_EE.stl" scale="0.001 0.001 0.001"/>
+          <mesh filename="file://$(find annin_ar4_description)/meshes/ar4_mk3/spraygun_EE.stl"
+                scale="0.001 0.001 0.001"/>
         </geometry>
       </collision>
