Commit message: Update ar_gripper_macro.srdf.xacro

File: annin_ar4_moveit_config/srdf/ar_gripper_macro.srdf.xacro (robot description, xacro)
@@ -1,25 +1,9 @@
 <?xml version="1.0" ?>
-<!--This does not replace URDF, and is not an extension of URDF.
-    This is a format for representing semantic information about the robot structure.
-    A URDF file must exist for this robot as well, where the joints and the links that are referenced are defined
--->
 <robot xmlns:xacro="http://wiki.ros.org/xacro">
   <xacro:macro name="ar_gripper_srdf" params="tf_prefix">
     <group name="ar_gripper">
       <link name="${tf_prefix}gripper_base_link" />
-      <link name="${tf_prefix}gripper_jaw1_link" />
-      <link name="${tf_prefix}gripper_jaw2_link" />
-      <joint name="${tf_prefix}gripper_jaw1_joint" />
-      <passive_joint name="${tf_prefix}gripper_jaw2_joint" />
     </group>
-    <group_state name="open" group="ar_gripper">
-      <joint name="${tf_prefix}gripper_jaw1_joint" value="0.012" />
-    </group_state>
-    <group_state name="closed" group="ar_gripper">
-      <joint name="${tf_prefix}gripper_jaw1_joint" value="0.001" />
-    </group_state>
-    <disable_collisions link1="${tf_prefix}gripper_base_link" link2="${tf_prefix}gripper_jaw1_link" reason="Adjacent" />
-    <disable_collisions link1="${tf_prefix}gripper_base_link" link2="${tf_prefix}gripper_jaw2_link" reason="Adjacent" />
-    <disable_collisions link1="${tf_prefix}gripper_jaw1_link" link2="${tf_prefix}gripper_jaw2_link" reason="Default" />
+    <!-- jaw1_joint, jaw2_joint 関連はすべて削除 -->
     <disable_collisions link1="${tf_prefix}link_6" link2="${tf_prefix}gripper_base_link" reason="Adjacent" />
     <disable_collisions link1="${tf_prefix}link_5" link2="${tf_prefix}gripper_base_link" reason="Adjacent" />
